Commit message: poprawnie dzialajacy program

File: visualization/urdf/movable.urdf (robot description, URDF)
Before this commit: robot manipulator, 4 links, 3 joints
Links:
- link link_3: geometry visual box size=0.2 0.2 0.7
Joints:
- joint link2_to_link3: axis (none) -> 0 0 1

File: visualization/urdf/state.urdf (robot description, URDF)
Before this commit: robot manipulator, 4 links, 3 joints
Links:
- link link_3: geometry visual box size=0.2 0.2 0.7

Commit message: poprawnie dzialajacy program

File: visualization/urdf/movable.urdf (robot description, URDF)
Before this commit: robot manipulator, 4 links, 3 joints
Links:
- link link_3: geometry visual box size=0.2 0.2 1
Joints:
- joint link2_to_link3: axis 0 0 1 -> 1 0 0

Commit message: Update movable.urdf

File: visualization/urdf/movable.urdf (robot description, URDF)
Before this commit: robot manipulator, 4 links, 3 joints
Joints:
- joint link2_to_link3: axis 1 0 0 -> 0 0 1

Commit message: Update movable.urdf

File: visualization/urdf/movable.urdf (robot description, URDF)
Before this commit: robot manipulator, 4 links, 3 joints
Links:
- link link_3: geometry visual box size=0.7 0.2 0.2
