Commit message: movable do poprawy

File: visualization/urdf/state.urdf (robot description, URDF)
Before this commit: robot manipulator, 4 links, 3 joints
Links:
- link link_3: geometry visual cylinder length=0.7 radius=0.06

Commit message: Update state.urdf

File: visualization/urdf/state.urdf (robot description, URDF)
Before this commit: robot manipulator, 4 links, 3 joints
Links:
- link link_3: geometry visual box size=0.7 0.2 0.2
Joints:
- joint link2_to_link3: axis (none) -> 0 0 1; limit (none) -> lower=0 upper=0.2 effort=1000.0 velocity=0.5; type fixed -> prismatic

Commit message: Update state.urdf

File: visualization/urdf/state.urdf (robot description, URDF)
Before this commit: robot manipulator, 4 links, 3 joints
Joints:
- joint link2_to_link3: type prismatic -> fixed
