Commit message: poprawnie zdzialajacy program

File: simple_kinematic/urdf/movable.urdf (robot description, URDF)
Before this commit: robot manipulator, 4 links, 3 joints
Joints:
- joint link2_to_link3: limit lower=0 upper=0.2 effort=1000.0 velocity=0.5 -> (none); type prismatic -> fixed

File: simple_kinematic/urdf/state.urdf (robot description, URDF)
Before this commit: robot manipulator, 4 links, 3 joints
Joints:
- joint base_to_link1: type continuous -> fixed
- joint link1_to_link2: limit lower=-1.57075 upper=1.57075 effort=1000.0 velocity=0.5 -> (none); type revolute -> fixed
- joint link2_to_link3: axis 0 0 1 -> (none); limit lower=0 upper=0.2 effort=1000.0 velocity=0.5 -> (none); type prismatic -> fixed

Commit message: poprawiony ostatni czlon

File: simple_kinematic/urdf/movable.urdf (robot description, URDF)
Before this commit: robot manipulator, 4 links, 3 joints
Links:
- link link_3: geometry visual box size=0.7 0.2 0.2
Joints:
- joint link2_to_link3: limit (none) -> lower=0 upper=0.2 effort=1000.0 velocity=0.5; type fixed -> prismatic

File: visualization/urdf/movable.urdf (robot description, URDF)
Before this commit: robot manipulator, 4 links, 3 joints
Links:
- link link_3: geometry visual box size=0.7 0.2 0.2
Joints:
- joint link2_to_link3: axis 1 0 0 -> 0 0 1

File: visualization/urdf/state.urdf (robot description, URDF)
Before this commit: robot manipulator, 4 links, 3 joints
Links:
- link link_3: geometry visual box size=0.7 0.2 0.2

Commit message: Poprawnie dzialajacy program

File: simple_kinematic/urdf/movable.urdf (robot description, URDF)
Before this commit: robot manipulator, 4 links, 3 joints
Joints:
- joint link1_to_link2: limit lower=-1.57075 upper=1.57075 effort=1000.0 velocity=0.5 -> lower=-2.57075 upper=2.57075 effort=1000.0 velocity=0.5
- joint link2_to_link3: limit lower=0 upper=0.2 effort=1000.0 velocity=0.5 -> lower=0 upper=0.35 effort=1000.0 velocity=0.5

Commit message: Last version

File: simple_kinematic/urdf/movable.urdf (robot description, URDF)
Before this commit: robot manipulator, 4 links, 3 joints
Joints:
- removed joint base_to_link1
- added joint base_link_to_link1: type continuous, parent base_link, child link_1, origin xyz=${props['i1']['j_xyz']} rpy=${props['i1']['j_rpy']}, axis 0 0 1
